File: arduino_duo_shield/arduino_duo_shield.sch (KiCad schematic (older format))
At the start: 17 parts, among them J2 EStop, J3 Motor_Control, J4 Limit_Switches, J5 inverter_freq, J6 inverter_cmd, J8 inverter_power, J9 Motor_Control_Mirror, P10 Digital, P11 PWM, P12 PWM, P13 Communication, P7 Power, P8 Analog, P9 Analog, SW1 SW_Push

Commit message: Added screw connectors to everything
Parts:
- removed J2: EStop, TerminalBlock:TerminalBlock_bornier-2_P5.08mm, symbol Connector:Conn_01x02_Female
- removed J3: Motor_Control, Connector_PinHeader_2.54mm:PinHeader_2x12_P2.54mm_Vertical, symbol Connector_Generic:Conn_02x12_Odd_Even
- removed J4: Limit_Switches, Connector_PinHeader_2.54mm:PinHeader_2x09_P2.54mm_Vertical, symbol Connector_Generic:Conn_01x18
- removed J5: inverter_freq, TerminalBlock:TerminalBlock_bornier-2_P5.08mm, symbol Connector:Conn_01x02_Male
- removed J6: inverter_cmd, TerminalBlock:TerminalBlock_bornier-2_P5.08mm, symbol Connector:Conn_01x02_Male
- removed J8: inverter_power, TerminalBlock:TerminalBlock_bornier-2_P5.08mm, symbol Connector:Conn_01x02_Male
- removed J9: Motor_Control_Mirror, Connector_PinHeader_2.54mm:PinHeader_2x12_P2.54mm_Vertical, symbol Connector_Generic:Conn_02x12_Odd_Even
- added J1: Limit_XY, Connectors:SCREWTERMINAL-3.5MM-4, symbol Connector:Screw_Terminal_01x04
- added J10: Inverter_Analog, Connectors:SCREWTERMINAL-3.5MM-2, symbol Connector:Screw_Terminal_01x02
- added J11: Inverter_Direction, Connectors:SCREWTERMINAL-3.5MM-2, symbol Connector:Screw_Terminal_01x02
- added J12: Inverter_12V, Connectors:SCREWTERMINAL-3.5MM-2, symbol Connector:Screw_Terminal_01x02
- added J13: EStop, Connectors:SCREWTERMINAL-3.5MM-2, symbol Connector:Screw_Terminal_01x02
- added J14: M1, Connectors:SCREWTERMINAL-3.5MM-3, symbol Connector:Screw_Terminal_01x03
- added J15: M2, Connectors:SCREWTERMINAL-3.5MM-3, symbol Connector:Screw_Terminal_01x03
- added J16: M3, Connectors:SCREWTERMINAL-3.5MM-3, symbol Connector:Screw_Terminal_01x03
- added J17: M4, Connectors:SCREWTERMINAL-3.5MM-3, symbol Connector:Screw_Terminal_01x03
- added J18: GND, Connectors:SCREWTERMINAL-3.5MM-2, symbol Connector:Screw_Terminal_01x02
- added J2: Limit_COM, Connectors:SCREWTERMINAL-3.5MM-2, symbol Connector:Screw_Terminal_01x02
- added J3: Limit_ZA, Connectors:SCREWTERMINAL-3.5MM-4, symbol Connector:Screw_Terminal_01x04
- added J4: Probe, Connectors:SCREWTERMINAL-3.5MM-2, symbol Connector:Screw_Terminal_01x02
Connections:
- wire segments 276 -> 223
